File: hardware/plate_top/plate_top.kicad_pcb (KiCad board)
At the start: 2 copper layers, 16 x 16 mm, 0 parts

Commit message: Revert "update kicad 7"
This reverts commit 5275a3c603f42084073b311218bfcafc03e2b97c.
Other:
- net class Default added: clearance 0.2, trace_width 0.25, via_dia 0.8, via_drill 0.4
- net class PW added: clearance 0.2, trace_width 0.4, via_dia 0.8, via_drill 0.4
Changed lines of the file:
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@@
-(kicad_pcb (version 20221018) (generator pcbnew)
+(kicad_pcb (version 20171130) (host pcbnew "(5.1.6)-1")
   (general
     (thickness 1.6)
+    (drawings 13)
+    (tracks 0)
+    (zones 0)
+    (modules 0)
+    (nets 1)
   )
-  (paper "A4")
+  (page A4)
   (layers
-    (0 "F.Cu" signal)
-    (31 "B.Cu" signal)
-    (32 "B.Adhes" user "B.Adhesive")
-    (33 "F.Adhes" user "F.Adhesive")
-    (34 "B.Paste" user)
-    (35 "F.Paste" user)
-    (36 "B.SilkS" user "B.Silkscreen")
-    (37 "F.SilkS" user "F.Silkscreen")
-    (38 "B.Mask" user)
-    (39 "F.Mask" user)
-    (40 "Dwgs.User" user "User.Drawings")
-    (41 "Cmts.User" user "User.Comments")
-    (42 "Eco1.User" user "User.Eco1")
-    (43 "Eco2.User" user "User.Eco2")
-    (44 "Edge.Cuts" user)
-    (45 "Margin" user)
-    (46 "B.CrtYd" user "B.Courtyard")
-    (47 "F.CrtYd" user "F.Courtyard")
-    (48 "B.Fab" user)
-    (49 "F.Fab" user)
+    (0 F.Cu signal)
+    (31 B.Cu signal)
+    (32 B.Adhes user)
+    (33 F.Adhes user)
+    (34 B.Paste user)
+    (35 F.Paste user)
+    (36 B.SilkS user)
+    (37 F.SilkS user)
+    (38 B.Mask user)
+    (39 F.Mask user)
+    (40 Dwgs.User user)
+    (41 Cmts.User user)
+    (42 Eco1.User user)
+    (43 Eco2.User user)
+    (44 Edge.Cuts user)
+    (45 Margin user)
+    (46 B.CrtYd user)
+    (47 F.CrtYd user)
+    (48 B.Fab user)
+    (49 F.Fab user)
   )
   (setup
+    (last_trace_width 0.25)
+    (trace_clearance 0.2)
+    (zone_clearance 0.508)
+    (zone_45_only no)
+    (trace_min 0.2)
+    (via_size 0.8)
+    (via_drill 0.4)
+    (via_min_size 0.4)
+    (via_min_drill 0.3)
+    (uvia_size 0.3)
+    (uvia_drill 0.1)
+    (uvias_allowed no)
+    (uvia_min_size 0.2)
+    (uvia_min_drill 0.1)
+    (edge_width 0.05)
+    (segment_width 0.2)
+    (pcb_text_width 0.3)
+    (pcb_text_size 1.5 1.5)
+    (mod_edge_width 0.12)
+    (mod_text_size 1 1)
+    (mod_text_width 0.15)
+    (pad_size 0.9 0.9)
+    (pad_drill 0)
     (pad_to_mask_clearance 0.05)
     (aux_axis_origin 125 90)
     (grid_origin 125 90)
+    (visible_elements 7FFFFFFF)
     (pcbplotparams
-      (layerselection 0x00010fc_ffffffff)
-      (plot_on_all_layers_selection 0x0000000_00000000)
-      (disableapertmacros false)
+      (layerselection 0x010fc_ffffffff)
       (usegerberextensions false)
       (usegerberattributes true)
       (usegerberadvancedattributes true)
       (creategerberjobfile true)
-      (dashed_line_dash_ratio 12.000000)
-      (dashed_line_gap_ratio 3.000000)
-      (svgprecision 4)
+      (excludeedgelayer true)
+      (linewidth 0.150000)
       (plotframeref false)
       (viasonmask false)
@@
       (hpglpenspeed 20)
       (hpglpendiameter 15.000000)
-      (dxfpolygonmode true)
-      (dxfimperialunits true)
-      (dxfusepcbnewfont true)
       (psnegative false)
       (psa4output false)
@@
       (plotvalue true)
       (plotinvisibletext false)
-      (sketchpadsonfab false)
+      (padsonsilk false)
       (subtractmaskfromsilk false)
       (outputformat 5)
@@
       (drillshape 0)
       (scaleselection 1)
-      (outputdirectory "trackball_dip_13_plate/")
-    )
+      (outputdirectory "trackball_dip_13_plate/"))
   )
   (net 0 "")
-  (gr_line (start 133 96.5) (end 133 83.5)
-    (stroke (width 0.05) (type solid)) (layer "Edge.Cuts"))
-  (gr_arc (start 131.5 82) (mid 132.56066 82.43934) (end 133 83.5)
-    (stroke (width 0.05) (type solid)) (layer "Edge.Cuts"))
-  (gr_arc (start 117 83.5) (mid 117.43934 82.43934) (end 118.5 82)
-    (stroke (width 0.05) (type solid)) (layer "Edge.Cuts"))
-  (gr_line (start 118.5 98) (end 131.5 98)
-    (stroke (width 0.05) (type solid)) (layer "Edge.Cuts"))
-  (gr_arc (start 118.5 98) (mid 117.43934 97.56066) (end 117 96.5)
-    (stroke (width 0.05) (type solid)) (layer "Edge.Cuts"))
-  (gr_arc (start 133 96.5) (mid 132.56066 97.56066) (end 131.5 98)
-    (stroke (width 0.05) (type solid)) (layer "Edge.Cuts"))
-  (gr_line (start 117 83.5) (end 117 96.5)
-    (stroke (width 0.05) (type solid)) (layer "Edge.Cuts"))
-  (gr_line (start 131.5 82) (end 118.5 82)
-    (stroke (width 0.05) (type solid)) (layer "Edge.Cuts"))
-  (gr_circle (center 118.5 83.5) (end 119.35 83.5)
-    (stroke (width 0.05) (type solid)) (fill none) (layer "Edge.Cuts"))
-  (gr_circle (center 131.5 96.5) (end 132.35 96.5)
-    (stroke (width 0.05) (type solid)) (fill none) (layer "Edge.Cuts"))
-  (gr_circle (center 131.5 83.5) (end 132.35 83.5)
-    (stroke (width 0.05) (type solid)) (fill none) (layer "Edge.Cuts"))
-  (gr_circle (center 118.5 96.5) (end 119.35 96.5)
-    (stroke (width 0.05) (type solid)) (fill none) (layer "Edge.Cuts"))
-  (gr_circle (center 125 90) (end 128.6 90)
-    (stroke (width 0.05) (type solid)) (fill none) (layer "Edge.Cuts"))
+  (net_class Default "これはデフォルトのネット クラスです。"
+    (clearance 0.2)
+    (trace_width 0.25)
+    (via_dia 0.8)
+    (via_drill 0.4)
+    (uvia_dia 0.3)
+    (uvia_drill 0.1)
+  )
+  (net_class PW ""
+    (clearance 0.2)
+    (trace_width 0.4)
+    (via_dia 0.8)
+    (via_drill 0.4)
+    (uvia_dia 0.3)
+    (uvia_drill 0.1)
+  )
+  (gr_circle (center 118.5 83.5) (end 119.35 83.5) (layer Edge.Cuts) (width 0.05))
+  (gr_circle (center 131.5 96.5) (end 132.35 96.5) (layer Edge.Cuts) (width 0.05))
+  (gr_line (start 118.5 98) (end 131.5 98) (layer Edge.Cuts) (width 0.05))
+  (gr_circle (center 118.5 96.5) (end 119.35 96.5) (layer Edge.Cuts) (width 0.05))
+  (gr_arc (start 118.5 96.5) (end 117 96.5) (angle -90) (layer Edge.Cuts) (width 0.05))
+  (gr_arc (start 131.5 83.5) (end 133 83.5) (angle -90) (layer Edge.Cuts) (width 0.05))
+  (gr_arc (start 118.5 83.5) (end 118.5 82) (angle -90) (layer Edge.Cuts) (width 0.05))
+  (gr_arc (start 131.5 96.5) (end 131.5 98) (angle -90) (layer Edge.Cuts) (width 0.05))
+  (gr_line (start 131.5 82) (end 118.5 82) (layer Edge.Cuts) (width 0.05))
+  (gr_circle (center 131.5 83.5) (end 132.35 83.5) (layer Edge.Cuts) (width 0.05))
+  (gr_line (start 133 96.5) (end 133 83.5) (layer Edge.Cuts) (width 0.05))
+  (gr_line (start 117 83.5) (end 117 96.5) (layer Edge.Cuts) (width 0.05))
+  (gr_circle (center 125 90) (end 128.6 90) (layer Edge.Cuts) (width 0.05))
 )

Commit message: update kicad 7
Other:
- net class Default removed
- net class PW removed
Changed lines of the file:
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@@
-(kicad_pcb (version 20171130) (host pcbnew "(5.1.6)-1")
+(kicad_pcb (version 20221018) (generator pcbnew)
   (general
     (thickness 1.6)
-    (drawings 13)
-    (tracks 0)
-    (zones 0)
-    (modules 0)
-    (nets 1)
   )
-  (page A4)
+  (paper "A4")
   (layers
-    (0 F.Cu signal)
-    (31 B.Cu signal)
-    (32 B.Adhes user)
-    (33 F.Adhes user)
-    (34 B.Paste user)
-    (35 F.Paste user)
-    (36 B.SilkS user)
-    (37 F.SilkS user)
-    (38 B.Mask user)
-    (39 F.Mask user)
-    (40 Dwgs.User user)
-    (41 Cmts.User user)
-    (42 Eco1.User user)
-    (43 Eco2.User user)
-    (44 Edge.Cuts user)
-    (45 Margin user)
-    (46 B.CrtYd user)
-    (47 F.CrtYd user)
-    (48 B.Fab user)
-    (49 F.Fab user)
+    (0 "F.Cu" signal)
+    (31 "B.Cu" signal)
+    (32 "B.Adhes" user "B.Adhesive")
+    (33 "F.Adhes" user "F.Adhesive")
+    (34 "B.Paste" user)
+    (35 "F.Paste" user)
+    (36 "B.SilkS" user "B.Silkscreen")
+    (37 "F.SilkS" user "F.Silkscreen")
+    (38 "B.Mask" user)
+    (39 "F.Mask" user)
+    (40 "Dwgs.User" user "User.Drawings")
+    (41 "Cmts.User" user "User.Comments")
+    (42 "Eco1.User" user "User.Eco1")
+    (43 "Eco2.User" user "User.Eco2")
+    (44 "Edge.Cuts" user)
+    (45 "Margin" user)
+    (46 "B.CrtYd" user "B.Courtyard")
+    (47 "F.CrtYd" user "F.Courtyard")
+    (48 "B.Fab" user)
+    (49 "F.Fab" user)
   )
   (setup
-    (last_trace_width 0.25)
-    (trace_clearance 0.2)
-    (zone_clearance 0.508)
-    (zone_45_only no)
-    (trace_min 0.2)
-    (via_size 0.8)
-    (via_drill 0.4)
-    (via_min_size 0.4)
-    (via_min_drill 0.3)
-    (uvia_size 0.3)
-    (uvia_drill 0.1)
-    (uvias_allowed no)
-    (uvia_min_size 0.2)
-    (uvia_min_drill 0.1)
-    (edge_width 0.05)
-    (segment_width 0.2)
-    (pcb_text_width 0.3)
-    (pcb_text_size 1.5 1.5)
-    (mod_edge_width 0.12)
-    (mod_text_size 1 1)
-    (mod_text_width 0.15)
-    (pad_size 0.9 0.9)
-    (pad_drill 0)
     (pad_to_mask_clearance 0.05)
     (aux_axis_origin 125 90)
     (grid_origin 125 90)
-    (visible_elements 7FFFFFFF)
     (pcbplotparams
-      (layerselection 0x010fc_ffffffff)
+      (layerselection 0x00010fc_ffffffff)
+      (plot_on_all_layers_selection 0x0000000_00000000)
+      (disableapertmacros false)
       (usegerberextensions false)
       (usegerberattributes true)
       (usegerberadvancedattributes true)
       (creategerberjobfile true)
-      (excludeedgelayer true)
-      (linewidth 0.150000)
+      (dashed_line_dash_ratio 12.000000)
+      (dashed_line_gap_ratio 3.000000)
+      (svgprecision 4)
       (plotframeref false)
       (viasonmask false)
@@
       (hpglpenspeed 20)
       (hpglpendiameter 15.000000)
+      (dxfpolygonmode true)
+      (dxfimperialunits true)
+      (dxfusepcbnewfont true)
       (psnegative false)
       (psa4output false)
@@
       (plotvalue true)
       (plotinvisibletext false)
-      (padsonsilk false)
+      (sketchpadsonfab false)
       (subtractmaskfromsilk false)
       (outputformat 5)
@@
       (drillshape 0)
       (scaleselection 1)
-      (outputdirectory "trackball_dip_13_plate/"))
+      (outputdirectory "trackball_dip_13_plate/")
+    )
   )
   (net 0 "")
-  (net_class Default "これはデフォルトのネット クラスです。"
-    (clearance 0.2)
-    (trace_width 0.25)
-    (via_dia 0.8)
-    (via_drill 0.4)
-    (uvia_dia 0.3)
-    (uvia_drill 0.1)
-  )
-  (net_class PW ""
-    (clearance 0.2)
-    (trace_width 0.4)
-    (via_dia 0.8)
-    (via_drill 0.4)
-    (uvia_dia 0.3)
-    (uvia_drill 0.1)
-  )
-  (gr_circle (center 118.5 83.5) (end 119.35 83.5) (layer Edge.Cuts) (width 0.05))
-  (gr_circle (center 131.5 96.5) (end 132.35 96.5) (layer Edge.Cuts) (width 0.05))
-  (gr_line (start 118.5 98) (end 131.5 98) (layer Edge.Cuts) (width 0.05))
-  (gr_circle (center 118.5 96.5) (end 119.35 96.5) (layer Edge.Cuts) (width 0.05))
-  (gr_arc (start 118.5 96.5) (end 117 96.5) (angle -90) (layer Edge.Cuts) (width 0.05))
-  (gr_arc (start 131.5 83.5) (end 133 83.5) (angle -90) (layer Edge.Cuts) (width 0.05))
-  (gr_arc (start 118.5 83.5) (end 118.5 82) (angle -90) (layer Edge.Cuts) (width 0.05))
-  (gr_arc (start 131.5 96.5) (end 131.5 98) (angle -90) (layer Edge.Cuts) (width 0.05))
-  (gr_line (start 131.5 82) (end 118.5 82) (layer Edge.Cuts) (width 0.05))
-  (gr_circle (center 131.5 83.5) (end 132.35 83.5) (layer Edge.Cuts) (width 0.05))
-  (gr_line (start 133 96.5) (end 133 83.5) (layer Edge.Cuts) (width 0.05))
-  (gr_line (start 117 83.5) (end 117 96.5) (layer Edge.Cuts) (width 0.05))
-  (gr_circle (center 125 90) (end 128.6 90) (layer Edge.Cuts) (width 0.05))
+  (gr_line (start 133 96.5) (end 133 83.5)
+    (stroke (width 0.05) (type solid)) (layer "Edge.Cuts"))
+  (gr_arc (start 131.5 82) (mid 132.56066 82.43934) (end 133 83.5)
+    (stroke (width 0.05) (type solid)) (layer "Edge.Cuts"))
+  (gr_arc (start 117 83.5) (mid 117.43934 82.43934) (end 118.5 82)
+    (stroke (width 0.05) (type solid)) (layer "Edge.Cuts"))
+  (gr_line (start 118.5 98) (end 131.5 98)
+    (stroke (width 0.05) (type solid)) (layer "Edge.Cuts"))
+  (gr_arc (start 118.5 98) (mid 117.43934 97.56066) (end 117 96.5)
+    (stroke (width 0.05) (type solid)) (layer "Edge.Cuts"))
+  (gr_arc (start 133 96.5) (mid 132.56066 97.56066) (end 131.5 98)
+    (stroke (width 0.05) (type solid)) (layer "Edge.Cuts"))
+  (gr_line (start 117 83.5) (end 117 96.5)
+    (stroke (width 0.05) (type solid)) (layer "Edge.Cuts"))
+  (gr_line (start 131.5 82) (end 118.5 82)
+    (stroke (width 0.05) (type solid)) (layer "Edge.Cuts"))
+  (gr_circle (center 118.5 83.5) (end 119.35 83.5)
+    (stroke (width 0.05) (type solid)) (fill none) (layer "Edge.Cuts"))
+  (gr_circle (center 131.5 96.5) (end 132.35 96.5)
+    (stroke (width 0.05) (type solid)) (fill none) (layer "Edge.Cuts"))
+  (gr_circle (center 131.5 83.5) (end 132.35 83.5)
+    (stroke (width 0.05) (type solid)) (fill none) (layer "Edge.Cuts"))
+  (gr_circle (center 118.5 96.5) (end 119.35 96.5)
+    (stroke (width 0.05) (type solid)) (fill none) (layer "Edge.Cuts"))
+  (gr_circle (center 125 90) (end 128.6 90)
+    (stroke (width 0.05) (type solid)) (fill none) (layer "Edge.Cuts"))
 )
